File: keyboard.kicad_pcb (KiCad board)
At the start: 2 copper layers, 21 parts, among them SW1 SW_SPST, SW10 SW_SPST, SW11 SW_SPST, SW12 SW_SPST, SW13 SW_SPST, SW14 SW_SPST, SW15 SW_SPST, SW16 SW_SPST, SW17 SW_SPST, SW18 SW_SPST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

Commit message: pcb
Parts:
- added D1: D, Diode_THT:D_T-1_P5.08mm_Horizontal, F.Cu at (48.1, 72.9)
- added D10: D, Diode_THT:D_T-1_P5.08mm_Horizontal, F.Cu at (56.8, 81.2)
- added D11: D, Diode_THT:D_T-1_P5.08mm_Horizontal, F.Cu at (56.8, 85.3)
- added D12: D, Diode_THT:D_T-1_P5.08mm_Horizontal, F.Cu at (56.8, 89.5)
- added D13: D, Diode_THT:D_T-1_P5.08mm_Horizontal, F.Cu at (56.8, 93.7)
- added D14: D, Diode_THT:D_T-1_P5.08mm_Horizontal, F.Cu at (56.8, 97.8)
- added D15: D, Diode_THT:D_T-1_P5.08mm_Horizontal, F.Cu at (38.9, 73.4)
- added D16: D, Diode_THT:D_T-1_P5.08mm_Horizontal, F.Cu at (43.7, 64.4)
- added D17: D, Diode_THT:D_T-1_P5.08mm_Horizontal, F.Cu at (38.9, 81.7)
- added D18: D, Diode_THT:D_T-1_P5.08mm_Horizontal, F.Cu at (38.9, 85.9)
- added D19: D, Diode_THT:D_T-1_P5.08mm_Horizontal, F.Cu at (38.9, 90.0)
- added D2: D, Diode_THT:D_T-1_P5.08mm_Horizontal, F.Cu at (48.1, 77.0)
- added D20: D, Diode_THT:D_T-1_P5.08mm_Horizontal, F.Cu at (38.9, 94.2)
- added D3: D, Diode_THT:D_T-1_P5.08mm_Horizontal, F.Cu at (48.1, 81.2)
- added D4: D, Diode_THT:D_T-1_P5.08mm_Horizontal, F.Cu at (48.1, 85.3)
- added D5: D, Diode_THT:D_T-1_P5.08mm_Horizontal, F.Cu at (48.1, 89.5)
- added D6: D, Diode_THT:D_T-1_P5.08mm_Horizontal, F.Cu at (48.1, 93.7)
- added D7: D, Diode_THT:D_T-1_P5.08mm_Horizontal, F.Cu at (48.1, 97.8)
- added D8: D, Diode_THT:D_T-1_P5.08mm_Horizontal, F.Cu at (56.8, 72.9)
- added D9: D, Diode_THT:D_T-1_P5.08mm_Horizontal, F.Cu at (56.8, 77.0)
- SW1, SW10, SW11, SW12, SW13, SW14, SW15, SW16, SW17, SW18, SW19, SW2, SW20, SW3, SW4, SW5, SW6, SW7, SW8, SW9: footprint Button_Switch_Keyboard:SW_Cherry_MX_1.00u_Plate -> PCM_Switch_Keyboard_Cherry_MX:SW_Cherry_MX_PCB
- moved SW17 74.1 mm to (168.8, 120.7)
- moved SW13 73.9 mm to (168.8, 101.2)
- moved SW9 73.7 mm to (168.8, 81.8)
- moved SW5 73.5 mm to (168.8, 62.3)
- moved SW1 73.4 mm to (168.8, 42.8)
- moved SW18 73.4 mm to (188.3, 120.7)
- moved SW14 73.2 mm to (188.3, 101.2)
- moved SW10 73.1 mm to (188.3, 81.8)
- moved SW6 72.8 mm to (188.3, 62.3)
- moved SW19 72.8 mm to (207.8, 120.7)
- moved SW2 72.8 mm to (188.3, 42.8)
- moved SW15 72.6 mm to (207.8, 101.2)
- moved SW11 72.4 mm to (207.8, 81.8)
- moved SW7 72.2 mm to (207.8, 62.3)
- moved SW3 72.1 mm to (207.8, 42.8)
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Connections:
- A1 pad 1: Net-(A1-Pad1) -> (no net)
- A1 pad 10: Net-(A1-Pad10) -> (no net)
- A1 pad 11: Net-(A1-Pad11) -> (no net)
- A1 pad 12: Net-(A1-Pad12) -> (no net)
- A1 pad 13: Net-(A1-Pad13) -> (no net)
- A1 pad 14: Net-(A1-Pad14) -> (no net)
- A1 pad 15: Net-(A1-Pad15) -> (no net)
- A1 pad 16: Net-(A1-Pad16) -> (no net)
- A1 pad 17: Net-(A1-Pad17) -> (no net)
- A1 pad 18: Net-(A1-Pad18) -> (no net)
- A1 pad 19: Net-(A1-Pad19) -> (no net)
- A1 pad 2: Net-(A1-Pad2) -> (no net)
- A1 pad 20: Net-(A1-Pad20) -> (no net)
- A1 pad 21: Net-(A1-Pad21) -> (no net)
- A1 pad 22: Net-(A1-Pad22) -> (no net)
- A1 pad 23: Net-(A1-Pad23) -> (no net)
- A1 pad 24: Net-(A1-Pad24) -> (no net)
- A1 pad 25: Net-(A1-Pad25) -> (no net)
- A1 pad 26: Net-(A1-Pad26) -> (no net)
- A1 pad 27: Net-(A1-Pad27) -> (no net)
- A1 pad 28: Net-(A1-Pad28) -> (no net)
- A1 pad 29: Net-(A1-Pad29) -> (no net)
- A1 pad 3: Net-(A1-Pad3) -> (no net)
- A1 pad 30: Net-(A1-Pad30) -> (no net)
- A1 pad 4: Net-(A1-Pad4) -> (no net)
- A1 pad 5: Net-(A1-Pad5) -> (no net)
- A1 pad 6: Net-(A1-Pad6) -> (no net)
- A1 pad 7: Net-(A1-Pad7) -> (no net)
- A1 pad 8: Net-(A1-Pad8) -> (no net)
- A1 pad 9: Net-(A1-Pad9) -> (no net)
- SW1 pad 1: Net-(SW1-Pad1) -> (no net)
- SW10 pad 1: Net-(SW10-Pad1) -> Net-(SW10-A)
- SW11 pad 1: Net-(SW10-Pad1) -> Net-(SW10-A)
- SW12 pad 1: Net-(SW10-Pad1) -> Net-(SW10-A)
- SW13 pad 1: Net-(SW13-Pad1) -> (no net)
- SW14 pad 1: Net-(SW13-Pad1) -> Net-(SW13-A)
- SW15 pad 1: Net-(SW13-Pad1) -> Net-(SW13-A)
- SW16 pad 1: Net-(SW13-Pad1) -> Net-(SW13-A)
- SW17 pad 1: Net-(SW17-Pad1) -> (no net)
- SW18 pad 1: Net-(SW17-Pad1) -> Net-(SW17-A)
- SW19 pad 1: Net-(SW17-Pad1) -> Net-(SW17-A)
- SW2 pad 1: Net-(SW1-Pad1) -> Net-(SW1-A)
- SW20 pad 1: Net-(SW17-Pad1) -> Net-(SW17-A)
- SW3 pad 1: Net-(SW1-Pad1) -> Net-(SW1-A)
- SW4 pad 1: Net-(SW1-Pad1) -> Net-(SW1-A)
- SW5 pad 1: Net-(SW5-Pad1) -> (no net)
- SW6 pad 1: Net-(SW5-Pad1) -> Net-(SW5-A)
- SW7 pad 1: Net-(SW5-Pad1) -> Net-(SW5-A)
- SW8 pad 1: Net-(SW5-Pad1) -> Net-(SW5-A)
- SW9 pad 1: Net-(SW10-Pad1) -> (no net)
Routing:
- net Net-(SW17-Pad1): track 61.3 -> 0.00 mm
- net Net-(SW13-Pad1): track 61.2 -> 0.00 mm
- net Net-(SW10-Pad1): track 61.2 -> 0.00 mm
- net Net-(SW5-Pad1): track 61.1 -> 0.04 mm
- net Net-(SW1-Pad1): track 61.1 -> 0.03 mm
Other:
- net class Default removed
